File: hardware/ReflowOven.sch (KiCad schematic (older format))
At the start: 41 parts

Commit message: Upgraded Files to latest Kicad 5
Parts:
- C? (x8): symbol C -> Device:C
- C? (x3): symbol CP1 -> Device:CP1
- D? (x2): symbol LED -> ReflowOven-rescue:LED
- D?: symbol D -> Device:D
- P?: symbol USB_B -> ReflowOven-rescue:USB_B
- P? (x3): symbol CONN_01X02 -> ReflowOven-rescue:CONN_01X02
- P?: symbol CONN_02X03 -> ReflowOven-rescue:CONN_02X03
- P?: symbol CONN_02X02 -> ReflowOven-rescue:CONN_02X02
- Q?: symbol Q_NMOS_SGD -> Device:Q_NMOS_SGD
- R? (x11): symbol Resistor -> ReflowOven-rescue:Resistor
- SW?: symbol SW_PUSH -> ReflowOven-rescue:SW_PUSH
- U?: symbol ATTINY84A-P -> ReflowOven-rescue:ATTINY84A-P
- U?: symbol MOC3041M -> ReflowOven-rescue:MOC3041M
- U?: symbol TRIAC -> ReflowOven-rescue:TRIAC
- U?: symbol FT232RL -> ReflowOven-rescue:FT232RL
- U?: symbol MAX31855 -> ReflowOven-rescue:MAX31855
- U?: symbol LM317T -> ReflowOven-rescue:LM317T
- VR? (x2): symbol VR -> ReflowOven-rescue:VR
